Commit message: xechayjduocroinmachinhthemhit

File: src/vacuum_driver/urdf/vacuum_robot.urdf (robot description, URDF)
Before this commit: robot vacuum_robot, 6 links, 5 joints
Links:
- link base_link: geometry collision box size=0.35 0.42 0.06; visual box size=0.35 0.42 0.06

Commit message: suacaitruc

File: src/vacuum_driver/urdf/vacuum_robot.urdf (robot description, URDF)
Before this commit: robot vacuum_robot, 6 links, 5 joints
Joints:
- joint base_to_laser: origin xyz=-0.10 0 0.081 rpy=0 0 0 -> xyz=0.10 0 0.081 rpy=0 0 0

Commit message: Rotate lidar frame 180 degrees

File: src/vacuum_driver/urdf/vacuum_robot.urdf (robot description, URDF)
Before this commit: robot vacuum_robot, 6 links, 5 joints
Joints:
- joint base_to_laser: origin xyz=0.10 0 0.081 rpy=0 0 0 -> xyz=0.10 0 0.081 rpy=0 0 3.14159265359

Commit message: rviz2 quay nguoc

File: src/vacuum_driver/urdf/vacuum_robot.urdf (robot description, URDF)
Before this commit: robot vacuum_robot, 6 links, 5 joints
Joints:
- joint base_to_laser: origin xyz=0.10 0 0.081 rpy=0 0 3.14159265359 -> xyz=-0.10 0 0.081 rpy=0 0 3.14159265359
